Commit message: Replace elbow link with strengthened native assembly and update renders

File: Simulation/PingTi_Arm_v4_new_calib/pingti_arm_v4_new_calib.urdf (robot description, URDF)
Before this commit: robot pingti_arm_v4_new_calib, 17 links, 16 joints
Links:
- link elbow_link: mass 0.09775001089453 -> 0.2008101791911
